File: KiCAD/ir2130_driver/ir2130_driver.kicad_pcb (KiCad board)
At the start: 2 copper layers, 90.3 x 113.9 mm, 26 parts, among them J1 Power Input, J2 Input, J3 Motor Output, Q1 IRFZ 24N, Q2 IRFZ 24N, Q3 IRFZ 24N, Q4 IRFZ 24N, Q5 IRFZ 24N, Q6 IRFZ 24N, U1 IR2130

Commit message: Added a standalone schematic for the STM32 part Moved from ir2130 driver to the TMC6140
Parts:
- J1: footprint Connector:Banana_Jack_2Pin -> TerminalBlock:TerminalBlock_bornier-2_P5.08mm
- J3: footprint Connector:Banana_Jack_3Pin -> TerminalBlock:TerminalBlock_Altech_AK300-3_P5.00mm
- moved J1 12.8 mm to (143.4, 47.8)
Routing:
- net V: track 163.7 -> 159.6 mm
- net +BATT: track 309.6 -> 310.7 mm
- net U: track 161.0 -> 161.8 mm
