File: KiCAD/ir2130_driver/ir2130_driver.kicad_sch (KiCad schematic)
At the start: 26 parts

Commit message: Added PCB file for the IR2130 test board
Parts:
- gave numbers to parts that had none: 26
Connections:
- net H2: now also J2.6 (Pin_6); no longer J2.5 (Pin_5)
- net H3: now also J2.5 (Pin_5); no longer J2.3 (Pin_3)
- net L1: now also J2.4 (Pin_4); no longer J2.6 (Pin_6)
- net L2: now also J2.3 (Pin_3); no longer J2.4 (Pin_4)
- net U: now also C4.2, U1.26 (VS1)
- net V: now also C5.2, U1.22 (VS2)
- net W: now also C6.2, U1.18 (VS3)

Commit message: Added a standalone schematic for the STM32 part Moved from ir2130 driver to the TMC6140
Parts:
- J1: footprint Connector:Banana_Jack_2Pin -> TerminalBlock:TerminalBlock_bornier-2_P5.08mm
- J3: footprint Connector:Banana_Jack_3Pin -> TerminalBlock:TerminalBlock_Altech_AK300-3_P5.00mm
Changed lines of the file:
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@@
     (property "Reference" "J1" (id 0) (at 38.1 58.5302 0))
     (property "Value" "Power Input" (id 1) (at 38.1 61.0671 0))
-    (property "Footprint" "Connector:Banana_Jack_2Pin" (id 2) (at 38.1 66.04 0)
+    (property "Footprint" "TerminalBlock:TerminalBlock_bornier-2_P5.08mm" (id 2) (at 38.1 66.04 0)
       (effects (font (size 1.27 1.27)) hide)
     )
@@
     (property "Reference" "J3" (id 0) (at 38.1 113.1402 0))
     (property "Value" "Motor Output" (id 1) (at 38.1 115.6771 0))
-    (property "Footprint" "Connector:Banana_Jack_3Pin" (id 2) (at 38.1 120.65 0)
+    (property "Footprint" "TerminalBlock:TerminalBlock_Altech_AK300-3_P5.00mm" (id 2) (at 38.1 120.65 0)
       (effects (font (size 1.27 1.27)) hide)
     )
@@
     )
     (path "/11675638-8398-443c-9cc4-596eff2ee906"
-      (reference "J1") (unit 1) (value "Power Input") (footprint "Connector:Banana_Jack_2Pin")
+      (reference "J1") (unit 1) (value "Power Input") (footprint "TerminalBlock:TerminalBlock_bornier-2_P5.08mm")
     )
     (path "/c52f6ce8-555a-42c7-a48b-4d6724c1e678"
@@
     )
     (path "/33b3b8c2-513d-40d4-ab04-6a367d51800d"
-      (reference "J3") (unit 1) (value "Motor Output") (footprint "Connector:Banana_Jack_3Pin")
+      (reference "J3") (unit 1) (value "Motor Output") (footprint "TerminalBlock:TerminalBlock_Altech_AK300-3_P5.00mm")
     )
     (path "/35d7a10e-09aa-4e19-80b9-d819f7adc131"
